File: fsae_daughterboard/fsae_daughterboard.kicad_sch (KiCad schematic)
At the start: 0 parts

Commit message: finished product
Parts:
- added C12, C13, C14: 100n, Capacitor_SMD:C_0805_2012Metric, symbol Device:C
- added J6: Conn_02x04_Odd_Even, Connector_Molex:Molex_Micro-Fit_3.0_43045-0812_2x04_P3.00mm_Vertical, symbol Connector_Generic:Conn_02x04_Odd_Even
- added LED3, LED4, LED5: LED, LED_THT:LED_D5.0mm, symbol Device:LED
- added R10, R8, R9: 10k, Resistor_SMD:R_0805_2012Metric, symbol Device:R
- added R5, R6, R7: 330, Resistor_SMD:R_0805_2012Metric, symbol Device:R
- added SW1, SW2, SW3: SW_Push, Button_Switch_THT:SW_PUSH_6mm_H5mm, symbol Switch:SW_Push
Connections:
- new net: LED4.2 (A), R6.2
- new net: LED5.2 (A), R7.2
- new net: LED3.2 (A), R5.2
- new net +3V3: J6.7 (Pin_7), R10.2, R8.2, R9.2
- new net BTN1: C12.1, J6.4 (Pin_4), R8.1, SW1.1
- new net BTN2: C13.1, J6.5 (Pin_5), R9.1, SW2.1
- new net BTN3: C14.1, J6.6 (Pin_6), R10.1, SW3.1
- new net GND: C12.2, C13.2, C14.2, J6.8 (Pin_8), LED3.1 (K), LED4.1 (K), LED5.1 (K), SW1.2, SW2.2, SW3.2
- new net LED_DB1: J6.1 (Pin_1), R5.1
- new net LED_DB2: J6.2 (Pin_2), R6.1
- new net LED_DB3: J6.3 (Pin_3), R7.1
